Commit message: modify joint state of plow and conveyor

File: bixi_description/urdf/accessories/conveyor.urdf.xacro (robot description, xacro)
@@ -4,49 +4,66 @@
     <xacro:property name="M_PI" value="3.1415926535897931"/>
     <!-- Base Size -->
+    <property name="conv_mass" value="1" />
     <property name="conv_x_size" value="0.7" />
     <property name="conv_y_size" value="0.22" />
-    <property name="conv_z_size" value="0.2" />
-    <property name="base_z_size" value="0.2" />
+    <property name="conv_z_size" value="0.02" />
+    <property name="base_z_size" value="0.1" />
     <link name="conveyor_link">
         <visual>
-            <origin xyz="0 0 0" rpy="0 0 0" />
+            <origin xyz="-${conv_x_size/2} 0 0" rpy="0 0 0" />
             <geometry>
-                <mesh filename="package://bixi_description/meshes/conveyor.dae" scale="0.01 0.01 0.01" />
+                <mesh filename="package://bixi_description/meshes/conveyor.dae" scale="1.64 3.28 3.28" />
             </geometry>
         </visual>
         <collision>
-            <origin xyz="0 0 0" rpy="0 0 0" />
+            <origin xyz="-${conv_x_size/2} 0 0" rpy="0 0 0" />
             <geometry>
-                <box size="${plow_x_size} ${plow_y_size} ${plow_z_size}"/>
+                <box size="${conv_x_size} ${conv_y_size} ${conv_z_size}"/>
             </geometry>
         </collision>
-        <!--collision>
-            <origin xyz="0 0 ${base_z_size*3/4}" rpy="0 0 0" />
-            <geometry>
-                <box size="${base_x_size*4/5} ${base_y_size} ${base_z_size/2}"/>
-            </geometry>
-        </collision-->
         <inertial>
-            <mass value="${base_mass}" />
+            <mass value="${conv_mass}" />
             <origin xyz="0 0 0" />
-            <inertia ixx="${1/12*base_mass*(base_x_size*base_x_size + base_z_size*base_z_size)}"
-                iyy="${1/12*base_mass*(base_y_size*base_y_size + base_z_size*base_z_size)}"
-                izz="${1/12*base_mass*(base_y_size*base_y_size + base_x_size*base_x_size)}"
+            <inertia ixx="${1/12*conv_mass*(conv_x_size*conv_x_size + conv_z_size*conv_z_size)}"
+                iyy="${1/12*conv_mass*(conv_y_size*conv_y_size + conv_z_size*conv_z_size)}"
+                izz="${1/12*conv_mass*(conv_y_size*conv_y_size + conv_x_size*conv_x_size)}"
                 ixy="0" ixz="0" iyz="0" />
         </inertial>
     </link>
     <link name="conveyor_extend_link">
+        <visual>
+            <origin xyz="-${conv_x_size/2} 0 0" rpy="0 0 0" />
+            <geometry>
+                <mesh filename="package://bixi_description/meshes/conveyor_extend.dae" scale="1.64 3.28 3.28" />
+            </geometry>
+        </visual>
+        <collision>
+            <origin xyz="-${conv_x_size/2} 0 0" rpy="0 0 0" />
+            <geometry>
+                <box size="${conv_x_size} ${conv_y_size} ${conv_z_size}"/>
+            </geometry>
+        </collision>
+        <inertial>
+            <mass value="${conv_mass}" />
+            <origin xyz="0 0 0" />
+            <inertia ixx="${1/12*conv_mass*(conv_x_size*conv_x_size + conv_z_size*conv_z_size)}"
+                iyy="${1/12*conv_mass*(conv_y_size*conv_y_size + conv_z_size*conv_z_size)}"
+                izz="${1/12*conv_mass*(conv_y_size*conv_y_size + conv_x_size*conv_x_size)}"
+                ixy="0" ixz="0" iyz="0" />
+        </inertial>
     </link>
     <joint name="conveyor_joint" type="revolute">
-        <origin xyz="0 0 0" rpy="0 0 0" />
+        <origin xyz="0.4 0 ${base_z_size+conv_z_size}" rpy="0 0 0" />
         <parent link="base_link" />
         <child link="conveyor_link" />
         <axis xyz="0 1 0" />
+        <limit lower="-0.15" upper="${M_PI/2}" effort="10" velocity="0.1" />
     </joint>
     <joint name="conveyor_extend_joint" type="prismatic">
-        <origin xyz="0 0 0" rpy="0 0 0" />
+        <origin xyz="-${conv_x_size/2} 0 0" rpy="0 0 0" />
         <parent link="conveyor_link" />
         <child link="conveyor_extend_link" />
         <axis xyz="-1 0 0" />
+        <limit lower="-0.35" upper="0.35" effort="10" velocity="0.1" />
     </joint>
 </robot>

File: bixi_description/urdf/accessories/plow.urdf.xacro (robot description, xacro)
@@ -4,13 +4,14 @@
     <xacro:property name="M_PI" value="3.1415926535897931"/>
     <!-- Base Size -->
+    <property name="plow_mass" value="0.2" />
     <property name="plow_x_size" value="0.02" />
     <property name="plow_y_size" value="0.45" />
     <property name="plow_z_size" value="0.2" />
     <property name="base_x_size" value="0.8" />
-<link name="plow_link">
-    <visual>
+    <link name="plow_link">
+        <visual>
             <origin xyz="0 0 0" rpy="0 0 0" />
             <geometry>
-                <mesh filename="package://bixi_description/meshes/plow.dae" scale="0.01 0.01 0.01" />
+                <mesh filename="package://bixi_description/meshes/plow.dae" scale="1 1 1" />
             </geometry>
         </visual>
@@ -21,21 +22,15 @@
             </geometry>
         </collision>
-        <!--collision>
-            <origin xyz="0 0 ${base_z_size*3/4}" rpy="0 0 0" />
-            <geometry>
-                <box size="${base_x_size*4/5} ${base_y_size} ${base_z_size/2}"/>
-            </geometry>
-        </collision-->
         <inertial>
-            <mass value="${base_mass}" />
+            <mass value="${plow_mass}" />
             <origin xyz="0 0 0" />
-            <inertia ixx="${1/12*base_mass*(base_x_size*base_x_size + base_z_size*base_z_size)}"
-                iyy="${1/12*base_mass*(base_y_size*base_y_size + base_z_size*base_z_size)}"
-                izz="${1/12*base_mass*(base_y_size*base_y_size + base_x_size*base_x_size)}"
+            <inertia ixx="${1/12*plow_mass*(plow_x_size*plow_x_size + plow_z_size*plow_z_size)}"
+                iyy="${1/12*plow_mass*(plow_y_size*plow_y_size + plow_z_size*plow_z_size)}"
+                izz="${1/12*plow_mass*(plow_y_size*plow_y_size + plow_x_size*plow_x_size)}"
                 ixy="0" ixz="0" iyz="0" />
         </inertial>
     </link>
     <joint name="plow_joint" type="fixed">
-        <origin xyz="0 ${base_x_size/2+plow_x_size/2} 0" rpy="0 0 0" />
+        <origin xyz="${base_x_size/2+plow_x_size/2} 0 0" rpy="0 0 0" />
         <parent link="base_link" />
         <child link="plow_link" />

File: bixi_description/urdf/standard.urdf.xacro (robot description, xacro)
@@ -7,4 +7,6 @@
     <xacro:include filename="materials.xacro" />
     <xacro:include filename="base.urdf.xacro" />
+    <xacro:include filename="accessories/plow.urdf.xacro" />
+    <xacro:include filename="accessories/conveyor.urdf.xacro" />
     <!--xacro:include filename="base.gazebo" />
     <xacro:include filename="sensor.urdf.xacro" />

Commit message: add conveor transmission for ros-control

File: bixi_description/urdf/accessories/conveyor.urdf.xacro (robot description, xacro)
@@ -67,3 +67,23 @@
         <limit lower="-0.35" upper="0.35" effort="10" velocity="0.1" />
     </joint>
+    <transmission name="tran_conveyor">
+        <type>transmission_interface/SimpleTransmission</type>
+        <joint name="conveyor_joint">
+            <hardwareInterface>EffortJointInterface</hardwareInterface>
+        </joint>
+        <actuator name="conveyor_motor">
+            <hardwareInterface>EffortJointInterface</hardwareInterface>
+            <mechanicalReduction>1</mechanicalReduction>
+        </actuator>
+    </transmission>
+    <transmission name="tran_conveyor_extend">
+        <type>transmission_interface/SimpleTransmission</type>
+        <joint name="conveyor_extend_joint">
+            <hardwareInterface>EffortJointInterface</hardwareInterface>
+        </joint>
+        <actuator name="conveyor_extend_motor">
+            <hardwareInterface>EffortJointInterface</hardwareInterface>
+            <mechanicalReduction>1</mechanicalReduction>
+        </actuator>
+    </transmission>
 </robot>

Commit message: fix visual scale mismatch

File: bixi_description/urdf/accessories/conveyor.urdf.xacro (robot description, xacro)
@@ -13,5 +13,5 @@
             <origin xyz="-${conv_x_size/2} 0 0" rpy="0 0 0" />
             <geometry>
-                <mesh filename="package://bixi_description/meshes/conveyor.dae" scale="1.64 3.28 3.28" />
+                <mesh filename="package://bixi_description/meshes/conveyor.dae" scale="3.28 3.28 3.28" />
             </geometry>
         </visual>
@@ -35,5 +35,5 @@
             <origin xyz="-${conv_x_size/2} 0 0" rpy="0 0 0" />
             <geometry>
-                <mesh filename="package://bixi_description/meshes/conveyor_extend.dae" scale="1.64 3.28 3.28" />
+                <mesh filename="package://bixi_description/meshes/conveyor_extend.dae" scale="3.28 3.28 3.28" />
             </geometry>
         </visual>
