Commit message: add dae and fix urdf bug

File: bixi_description/urdf/base.urdf.xacro (robot description, xacro)
@@ -1,8 +1,8 @@
 <?xml version="1.0"?>
 <!-- Revolute-Revolute Manipulator -->
-<robot name="robotx" xmlns:xacro="http://www.ros.org/wiki/xacro">
+<robot name="bixi" xmlns:xacro="http://www.ros.org/wiki/xacro">
     <xacro:include filename="$(find bixi_description)/urdf/wheel.urdf.xacro" />
     <!-- Constants for robot dimensions -->
-    <xacro:property name="PI" value="3.1415926535897931"/>
+    <xacro:property name="M_PI" value="3.1415926535897931"/>
     <!-- Base Size -->
     <property name="base_mass" value="10" />
@@ -20,47 +20,50 @@
     <!-- base link is the center of the robot's bottom plate -->
     <link name="base_link">
-      <visual>
-        <origin xyz="0 0 0" rpy="0 0 0" />
-        <geometry>
-          <mesh filename="package://bixi_description/meshes/chasis.dae" />
-        </geometry>
-      </visual>
-      <collision>
-        <origin xyz="0 0 ${base_z_size/4}" rpy="0 0 0" />
-        <geometry>
-          <box size="${base_x_size} ${base_y_size} ${base_z_size/2}"/>
-        </geometry>
-      </collision>
-      <collision>
-        <origin xyz="0 0 ${base_z_size*3/4}" rpy="0 0 0" />
-        <geometry>
-          <box size="${base_x_size*4/5} ${base_y_size} ${base_z_size/2}"/>
-        </geometry>
-      </collision>
-      <inertial>
-        <mass value="${base_mass}" />
-        <origin xyz="-0.08748 -0.00085 0.09947" />
-        <inertia ixx="0.6022" ixy="-0.02364" ixz="-0.1197" iyy="1.7386" iyz="-0.001544" izz="2.0296" />
-      </inertial>
+        <visual>
+            <origin xyz="0 0 0" rpy="0 0 0" />
+            <geometry>
+                <mesh filename="package://bixi_description/meshes/chasis.dae" scale="0.001 0.001 0.001" />
+            </geometry>
+        </visual>
+        <collision>
+            <origin xyz="0 0 0" rpy="0 0 0" />
+            <geometry>
+                <box size="${base_x_size} ${base_y_size} ${base_z_size}"/>
+            </geometry>
+        </collision>
+        <!--collision>
+            <origin xyz="0 0 ${base_z_size*3/4}" rpy="0 0 0" />
+            <geometry>
+                <box size="${base_x_size*4/5} ${base_y_size} ${base_z_size/2}"/>
+            </geometry>
+        </collision-->
+        <inertial>
+            <mass value="${base_mass}" />
+            <origin xyz="0 0 0" />
+            <inertia ixx="${1/12*base_mass*(base_x_size*base_x_size + base_z_size*base_z_size)}"
+                iyy="${1/12*base_mass*(base_y_size*base_y_size + base_z_size*base_z_size)}"
+                izz="${1/12*base_mass*(base_y_size*base_y_size + base_x_size*base_x_size)}"
+                ixy="0" ixz="0" iyz="0" />
+        </inertial>
     </link>
     <!-- Base footprint is on the ground under the robot -->
     <link name="base_footprint"/>
     <joint name="base_footprint_joint" type="fixed">
-      <origin xyz="0 0 ${wheel_vertical_offset - wheel_radius}" rpy="0 0 0" />
-      <parent link="base_link" />
-      <child link="base_footprint" />
+        <origin xyz="0 0 ${wheel_vertical_offset - wheel_radius}" rpy="0 0 0" />
+        <parent link="base_link" />
+        <child link="base_footprint" />
     </joint>
     <!-- Husky wheel macros -->
-    <xacro:wheel wheel_prefix="front_left">
-      <origin xyz="${wheelbase/2} ${track/2} ${wheel_vertical_offset}" rpy="0 0 0" />
+    <xacro:wheel ccw="1" wheel_prefix="front_left">
+        <origin xyz="${wheelbase/2} ${track/2} ${wheel_vertical_offset}" rpy="0 0 0" />
     </xacro:wheel>
-    <xacro:wheel wheel_prefix="front_right">
-      <origin xyz="${wheelbase/2} ${-track/2} ${wheel_vertical_offset}" rpy="0 0 0" />
+    <xacro:wheel ccw="0" wheel_prefix="front_right">
+        <origin xyz="${wheelbase/2} ${-track/2} ${wheel_vertical_offset}" rpy="0 0 0" />
     </xacro:wheel>
-    <xacro:wheel wheel_prefix="rear_left">
-      <origin xyz="${-wheelbase/2} ${track/2} ${wheel_vertical_offset}" rpy="0 0 0" />
+    <xacro:wheel ccw="1" wheel_prefix="rear_left">
+        <origin xyz="${-wheelbase/2} ${track/2} ${wheel_vertical_offset}" rpy="0 0 0" />
     </xacro:wheel>
-    <xacro:wheel wheel_prefix="rear_right">
-      <origin xyz="${-wheelbase/2} ${-track/2} ${wheel_vertical_offset}" rpy="0 0 0" />
+    <xacro:wheel ccw="0" wheel_prefix="rear_right">
+        <origin xyz="${-wheelbase/2} ${-track/2} ${wheel_vertical_offset}" rpy="0 0 0" />
     </xacro:wheel>
 </robot>

File: bixi_description/urdf/standard.urdf.xacro (robot description, xacro)
@@ -7,6 +7,6 @@
     <xacro:include filename="materials.xacro" />
     <xacro:include filename="base.urdf.xacro" />
-    <xacro:include filename="base.gazebo" />
+    <!--xacro:include filename="base.gazebo" />
     <xacro:include filename="sensor.urdf.xacro" />
-    <xacro:include filename="sensor.gazebo" />
+    <xacro:include filename="sensor.gazebo" /-->
 </robot>

File: bixi_description/urdf/wheel.urdf.xacro (robot description, xacro)
@@ -1,45 +1,59 @@
 <?xml version="1.0"?>
-<robot xmlns:xacro="http://ros.org/wiki/xacro" name="wheel">
-    <xacro:macro name="wheel" params="wheel_prefix *joint_pose">
-		<link name="${wheel_prefix}_wheel_link">
-			<inertial>
-				<mass value="${wheel_mass}" />
-				<origin xyz="0 0 0" />
-				<inertia  ixx="0.02467" ixy="0" ixz="0" iyy="0.04411" iyz="0" izz="0.02467" />
-			</inertial>
-			<visual>
-				<origin xyz="0 0 0" rpy="0 0 0" />
-				<geometry>
-					<mesh filename="package://bixi_description/meshes/wheel.dae" />
-				</geometry>
-			</visual>
-			<collision>
-				<origin xyz="0 0 0" rpy="${M_PI/2} 0 0" />
-				<geometry>
-					<cylinder length="${wheel_length}" radius="${wheel_radius}" />
-				</geometry>
-			</collision>
-		</link>
-		<gazebo reference="${wheel_prefix}_wheel_link">
-			<mu1 value="1.0"/>
-			<mu2 value="1.0"/>
-			<kp value="10000000.0" />
-			<kd value="1.0" />
-			<fdir1 value="1 0 0"/>
-		</gazebo>
-		<joint name="${wheel_prefix}_wheel" type="continuous">
-			<parent link="base_link"/>
-			<child link="${wheel_prefix}_wheel_link"/>
-			<xacro:insert_block name="joint_pose"/>
-			<axis xyz="0 1 0" rpy="0 0 0" />
-		</joint>
-		<transmission name="${wheel_prefix}_wheel_trans" type="SimpleTransmission">
-			<type>transmission_interface/SimpleTransmission</type>
-			<actuator name="${wheel_prefix}_wheel_motor">
-				<mechanicalReduction>1</mechanicalReduction>
-			</actuator>
-			<joint name="${wheel_prefix}_wheel">
-				<hardwareInterface>VelocityJointInterface</hardwareInterface>
-			</joint>
-		</transmission>
-	</xacro:macro>
+<robot xmlns:xacro="http://www.ros.org/wiki/xacro" name="wheel">
+    <!-- Wheel Properties -->
+    <xacro:property name="M_PI" value="3.1415926535897931"/>
+    <xacro:property name="wheel_mass" value="0.258" />
+    <xacro:property name="wheel_length" value="0.1143" />
+    <xacro:property name="wheel_radius" value="0.17775" />
+    <xacro:macro name="wheel" params="ccw wheel_prefix *joint_pose">
+        <link name="${wheel_prefix}_wheel_link">
+            <inertial>
+                <mass value="${wheel_mass}" />
+                <origin xyz="0 0 0" />
+                <inertia ixx="${1/12*wheel_mass*(3*wheel_radius*wheel_radius + wheel_length*wheel_length)}"
+                    iyy="${1/12*wheel_mass*(3*wheel_radius*wheel_radius + wheel_length*wheel_length)}"
+                    izz="${1/2*wheel_mass*wheel_radius*wheel_radius}"
+                    ixy="0" ixz="0" iyz="0" />
+            </inertial>
+            <visual>
+                <origin xyz="0 0 0" rpy="0 0 0" />
+                <geometry>
+                    <xacro:if value="${ccw == 1}">
+                    <mesh filename="package://bixi_description/meshes/mecanum_left.dae" scale="0.001 0.001 0.001"/>
+                </xacro:if>
+                    <xacro:if value="${ccw == 0}">
+                    <mesh filename="package://bixi_description/meshes/mecanum_right.dae" scale="0.001 0.001 0.001"/>
+                </xacro:if>
+                </geometry>
+            </visual>
+            <collision>
+                <origin xyz="0 0 0" rpy="${M_PI/2} 0 0" />
+                <geometry>
+                    <cylinder length="${wheel_length}" radius="${wheel_radius}" />
+                </geometry>
+            </collision>
+        </link>
+        <gazebo reference="${wheel_prefix}_wheel_link">
+            <mu1 value="1.0"/>
+            <mu2 value="1.0"/>
+            <kp value="10000000.0" />
+            <kd value="1.0" />
+            <fdir1 value="1 0 0"/>
+        </gazebo>
+        <joint name="${wheel_prefix}_wheel" type="continuous">
+            <parent link="base_link"/>
+            <child link="${wheel_prefix}_wheel_link"/>
+            <xacro:insert_block name="joint_pose"/>
+            <axis xyz="0 1 0" rpy="0 0 0" />
+        </joint>
+        <transmission name="${wheel_prefix}_wheel_trans" type="SimpleTransmission">
+            <type>transmission_interface/SimpleTransmission</type>
+            <actuator name="${wheel_prefix}_wheel_motor">
+                <mechanicalReduction>1</mechanicalReduction>
+            </actuator>
+            <joint name="${wheel_prefix}_wheel">
+                <hardwareInterface>VelocityJointInterface</hardwareInterface>
+            </joint>
+        </transmission>
+    </xacro:macro>
+</robot>

Commit message: modify wheel size, add plow

File: bixi_description/urdf/base.urdf.xacro (robot description, xacro)
@@ -7,15 +7,13 @@
     <!-- Base Size -->
     <property name="base_mass" value="10" />
-    <property name="base_x_size" value="0.98740000" />
-    <property name="base_y_size" value="0.57090000" />
-    <property name="base_z_size" value="0.24750000" />
+    <property name="base_x_size" value="0.8" />
+    <property name="base_y_size" value="0.4" />
+    <property name="base_z_size" value="0.1" />
     <!-- Wheel Mounting Positions -->
-    <xacro:property name="wheelbase" value="0.5120" />
-    <xacro:property name="track" value="0.5708" />
-    <xacro:property name="wheel_vertical_offset" value="0.03282" />
+    <xacro:property name="wheelbase" value="0.6" />
+    <xacro:property name="track" value="0.6" />
+    <xacro:property name="wheel_vertical_offset" value="0.05" />
     <!-- Wheel Properties -->
-    <xacro:property name="wheel_mass" value="0.258" />
-    <xacro:property name="wheel_length" value="0.1143" />
-    <xacro:property name="wheel_radius" value="0.17775" />
+    <xacro:property name="wheel_radius" value="0.075" />
     <!-- base link is the center of the robot's bottom plate -->
     <link name="base_link">
@@ -23,5 +21,5 @@
             <origin xyz="0 0 0" rpy="0 0 0" />
             <geometry>
-                <mesh filename="package://bixi_description/meshes/chasis.dae" scale="0.001 0.001 0.001" />
+                <mesh filename="package://bixi_description/meshes/chasis.dae" scale="1 1 1" />
             </geometry>
         </visual>
@@ -50,20 +48,20 @@
     <link name="base_footprint"/>
     <joint name="base_footprint_joint" type="fixed">
-        <origin xyz="0 0 ${wheel_vertical_offset - wheel_radius}" rpy="0 0 0" />
-        <parent link="base_link" />
-        <child link="base_footprint" />
+        <origin xyz="0 0 ${wheel_vertical_offset+wheel_radius}" rpy="0 0 0" />
+        <parent link="base_footprint" />
+        <child link="base_link" />
     </joint>
     <!-- Husky wheel macros -->
     <xacro:wheel ccw="1" wheel_prefix="front_left">
-        <origin xyz="${wheelbase/2} ${track/2} ${wheel_vertical_offset}" rpy="0 0 0" />
+        <origin xyz="${wheelbase/2} ${track/2} -${wheel_vertical_offset}" rpy="0 0 0" />
     </xacro:wheel>
     <xacro:wheel ccw="0" wheel_prefix="front_right">
-        <origin xyz="${wheelbase/2} ${-track/2} ${wheel_vertical_offset}" rpy="0 0 0" />
+        <origin xyz="${wheelbase/2} ${-track/2} -${wheel_vertical_offset}" rpy="0 0 0" />
     </xacro:wheel>
-    <xacro:wheel ccw="1" wheel_prefix="rear_left">
-        <origin xyz="${-wheelbase/2} ${track/2} ${wheel_vertical_offset}" rpy="0 0 0" />
+    <xacro:wheel ccw="0" wheel_prefix="rear_left">
+        <origin xyz="${-wheelbase/2} ${track/2} -${wheel_vertical_offset}" rpy="0 0 0" />
     </xacro:wheel>
-    <xacro:wheel ccw="0" wheel_prefix="rear_right">
-        <origin xyz="${-wheelbase/2} ${-track/2} ${wheel_vertical_offset}" rpy="0 0 0" />
+    <xacro:wheel ccw="1" wheel_prefix="rear_right">
+        <origin xyz="${-wheelbase/2} ${-track/2} -${wheel_vertical_offset}" rpy="0 0 0" />
     </xacro:wheel>
 </robot>

File: bixi_description/urdf/wheel.urdf.xacro (robot description, xacro)
@@ -3,7 +3,7 @@
     <!-- Wheel Properties -->
     <xacro:property name="M_PI" value="3.1415926535897931"/>
-    <xacro:property name="wheel_mass" value="0.258" />
-    <xacro:property name="wheel_length" value="0.1143" />
-    <xacro:property name="wheel_radius" value="0.17775" />
+    <xacro:property name="wheel_mass" value="0.158" />
+    <xacro:property name="wheel_length" value="0.02" />
+    <xacro:property name="wheel_radius" value="0.075" />
     <xacro:macro name="wheel" params="ccw wheel_prefix *joint_pose">
         <link name="${wheel_prefix}_wheel_link">
@@ -19,7 +19,7 @@
                 <origin xyz="0 0 0" rpy="0 0 0" />
                 <geometry>
-                    <xacro:if value="${ccw == 1}">
+                    <xacro:unless value="${ccw == 0}">
                     <mesh filename="package://bixi_description/meshes/mecanum_left.dae" scale="0.001 0.001 0.001"/>
-                </xacro:if>
+                </xacro:unless>
                     <xacro:if value="${ccw == 0}">
                     <mesh filename="package://bixi_description/meshes/mecanum_right.dae" scale="0.001 0.001 0.001"/>

Commit message: modify dae by sketchup to match dimension

File: bixi_description/urdf/base.urdf.xacro (robot description, xacro)
@@ -12,5 +12,5 @@
     <!-- Wheel Mounting Positions -->
     <xacro:property name="wheelbase" value="0.6" />
-    <xacro:property name="track" value="0.6" />
+    <xacro:property name="track" value="0.55" />
     <xacro:property name="wheel_vertical_offset" value="0.05" />
     <!-- Wheel Properties -->
@@ -30,10 +30,4 @@
             </geometry>
         </collision>
-        <!--collision>
-            <origin xyz="0 0 ${base_z_size*3/4}" rpy="0 0 0" />
-            <geometry>
-                <box size="${base_x_size*4/5} ${base_y_size} ${base_z_size/2}"/>
-            </geometry>
-        </collision-->
         <inertial>
             <mass value="${base_mass}" />

File: bixi_description/urdf/wheel.urdf.xacro (robot description, xacro)
@@ -4,5 +4,5 @@
     <xacro:property name="M_PI" value="3.1415926535897931"/>
     <xacro:property name="wheel_mass" value="0.158" />
-    <xacro:property name="wheel_length" value="0.02" />
+    <xacro:property name="wheel_length" value="0.05" />
     <xacro:property name="wheel_radius" value="0.075" />
     <xacro:macro name="wheel" params="ccw wheel_prefix *joint_pose">
@@ -20,9 +20,9 @@
                 <geometry>
                     <xacro:unless value="${ccw == 0}">
-                    <mesh filename="package://bixi_description/meshes/mecanum_left.dae" scale="0.001 0.001 0.001"/>
-                </xacro:unless>
+                        <mesh filename="package://bixi_description/meshes/mec_f_l.dae" scale="1 1 1"/>
+                    </xacro:unless>
                     <xacro:if value="${ccw == 0}">
-                    <mesh filename="package://bixi_description/meshes/mecanum_right.dae" scale="0.001 0.001 0.001"/>
-                </xacro:if>
+                        <mesh filename="package://bixi_description/meshes/mec_f_r.dae" scale="1 1 1"/>
+                    </xacro:if>
                 </geometry>
             </visual>

Commit message: modify urdf for adding sensor

File: bixi_description/urdf/base.urdf.xacro (robot description, xacro)
@@ -5,4 +5,5 @@
     <!-- Constants for robot dimensions -->
     <xacro:property name="M_PI" value="3.1415926535897931"/>
+    <!-- this section must be changed according to the real robot -->
     <!-- Base Size -->
     <property name="base_mass" value="10" />
@@ -39,5 +40,5 @@
         </inertial>
     </link>
-    <!-- Base footprint is on the ground under the robot -->
+    <!-- Base footprint is on the ground under the robot, NOT IN USE, use baselink as the root >
     <link name="base_footprint"/>
     <joint name="base_footprint_joint" type="fixed">
@@ -45,5 +46,5 @@
         <parent link="base_footprint" />
         <child link="base_link" />
-    </joint>
+    </joint -->
     <!-- Husky wheel macros -->
     <xacro:wheel ccw="1" wheel_prefix="front_left">

File: bixi_description/urdf/standard.urdf.xacro (robot description, xacro)
@@ -7,6 +7,8 @@
     <xacro:include filename="materials.xacro" />
     <xacro:include filename="base.urdf.xacro" />
+    <xacro:include filename="sensor.urdf.xacro" />
+    <!-- accessories >
     <xacro:include filename="accessories/plow.urdf.xacro" />
-    <xacro:include filename="accessories/conveyor.urdf.xacro" />
+    <xacro:include filename="accessories/conveyor.urdf.xacro" /-->
     <!--xacro:include filename="base.gazebo" />
     <xacro:include filename="sensor.urdf.xacro" />

File: bixi_description/urdf/wheel.urdf.xacro (robot description, xacro)
@@ -1,4 +1,5 @@
 <?xml version="1.0"?>
 <robot xmlns:xacro="http://www.ros.org/wiki/xacro" name="wheel">
+    <!-- this section must be changed according to the real robot -->
     <!-- Wheel Properties -->
     <xacro:property name="M_PI" value="3.1415926535897931"/>
